File: DingLAB_miniPC_Power_Vertical.kicad_sch (KiCad schematic)
At the start: 8 parts, among them J1 Conn_01x02_Pin, J2 Conn_01x02_Pin, U1 KJB48xxSBO-10A

Commit message: Update Vertical and product
Parts:
- H1, H2, H3: value MountingHole -> SMTSO3060CTJ; lcsc (none) -> C2915637
- R1: value 150k -> 20k
- R2: value 1.15M -> ∞
- U1: value KJB48xxSBO-10A -> KJB4815SBO-10A
Connections:
- net GND: now also R1.2, R2.1
- net Out: no longer R1.1, R2.1
- net at R2.2, U1.5 (Trim): now also R1.1; no longer R1.2
Other:
- moved on the sheet: R1, R2
Changed lines of the file:
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@@
   (junction (at 107.95 110.49) (diameter 0) (color 0 0 0 0)
   )
-  (junction (at 153.67 102.87) (diameter 0) (color 0 0 0 0)
-  )
   (junction (at 104.14 105.41) (diameter 0) (color 0 0 0 0)
   )
-  (junction (at 143.51 102.87) (diameter 0) (color 0 0 0 0)
-  )
-  (junction (at 143.51 110.49) (diameter 0) (color 0 0 0 0)
-  )
-  (wire (pts (xy 163.83 118.11) (xy 134.62 118.11))
-    (stroke (width 0) (type default))
+  (junction (at 143.51 118.11) (diameter 0) (color 0 0 0 0)
+  )
+  (junction (at 143.51 109.22) (diameter 0) (color 0 0 0 0)
+  )
+  (junction (at 153.67 118.11) (diameter 0) (color 0 0 0 0)
   )
   (wire (pts (xy 163.83 105.41) (xy 163.83 102.87))
     (stroke (width 0) (type default))
   )
-  (wire (pts (xy 138.43 110.49) (xy 143.51 110.49))
-    (stroke (width 0) (type default))
-  )
   (wire (pts (xy 133.35 106.68) (xy 138.43 106.68))
     (stroke (width 0) (type default))
@@
     (stroke (width 0) (type default))
   )
-  (wire (pts (xy 138.43 102.87) (xy 143.51 102.87))
-    (stroke (width 0) (type default))
-  )
   (wire (pts (xy 100.33 105.41) (xy 104.14 105.41))
     (stroke (width 0) (type default))
@@
     (stroke (width 0) (type default))
   )
+  (wire (pts (xy 143.51 109.22) (xy 153.67 109.22))
+    (stroke (width 0) (type default))
+  )
   (wire (pts (xy 138.43 106.68) (xy 138.43 104.14))
     (stroke (width 0) (type default))
   )
+  (wire (pts (xy 143.51 118.11) (xy 134.62 118.11))
+    (stroke (width 0) (type default))
+  )
   (wire (pts (xy 100.33 107.95) (xy 107.95 107.95))
     (stroke (width 0) (type default))
   )
-  (wire (pts (xy 133.35 109.22) (xy 138.43 109.22))
+  (wire (pts (xy 153.67 118.11) (xy 163.83 118.11))
+    (stroke (width 0) (type default))
+  )
+  (wire (pts (xy 153.67 116.84) (xy 153.67 118.11))
+    (stroke (width 0) (type default))
+  )
+  (wire (pts (xy 133.35 109.22) (xy 143.51 109.22))
     (stroke (width 0) (type default))
   )
@@
     (stroke (width 0) (type default))
   )
+  (wire (pts (xy 143.51 116.84) (xy 143.51 118.11))
+    (stroke (width 0) (type default))
+  )
   (wire (pts (xy 107.95 110.49) (xy 110.49 110.49))
     (stroke (width 0) (type default))
   )
-  (wire (pts (xy 143.51 102.87) (xy 153.67 102.87))
-    (stroke (width 0) (type default))
-  )
-  (wire (pts (xy 163.83 102.87) (xy 153.67 102.87))
+  (wire (pts (xy 138.43 102.87) (xy 163.83 102.87))
     (stroke (width 0) (type default))
   )
@@
     (stroke (width 0) (type default))
   )
+  (wire (pts (xy 153.67 118.11) (xy 143.51 118.11))
+    (stroke (width 0) (type default))
+  )
   (wire (pts (xy 138.43 104.14) (xy 138.43 102.87))
-    (stroke (width 0) (type default))
-  )
-  (wire (pts (xy 143.51 110.49) (xy 153.67 110.49))
-    (stroke (width 0) (type default))
-  )
-  (wire (pts (xy 138.43 109.22) (xy 138.43 110.49))
     (stroke (width 0) (type default))
   )
@@
         )
       )
-      (project "DingLAB_miniPC_Power"
+      (project "DingLAB_miniPC_Power_Vertical"
         (path "/b2cfdd7f-acce-42ad-aab6-fa699ca2dca8"
           (reference "J2") (unit 1)
@@
         )
       )
-      (project "DingLAB_miniPC_Power"
+      (project "DingLAB_miniPC_Power_Vertical"
         (path "/b2cfdd7f-acce-42ad-aab6-fa699ca2dca8"
           (reference "#PWR02") (unit 1)
@@
       (effects (font (size 1.27 1.27)) (justify left))
     )
-    (property "Value" "MountingHole" (at 129.54 147.32 0)
+    (property "Value" "SMTSO3060CTJ" (at 129.54 147.32 0)
       (effects (font (size 1.27 1.27)) (justify left))
     )
@@
       (effects (font (size 1.27 1.27)) hide)
     )
-    (instances
-      (project "DingLAB_miniPC_Power"
+    (property "lcsc" "C2915637" (at 127 146.05 0)
+      (effects (font (size 1.27 1.27)) hide)
+    )
+    (instances
+      (project "DingLAB_miniPC_Power_Vertical"
         (path "/b2cfdd7f-acce-42ad-aab6-fa699ca2dca8"
           (reference "H3") (unit 1)
@@
     )
   )
-  (symbol (lib_id "Device:R") (at 153.67 106.68 0) (unit 1)
-    (in_bom yes) (on_board yes) (dnp no) (fields_autoplaced)
-    (property "Reference" "R2" (at 156.21 105.41 0)
-      (effects (font (size 1.27 1.27)) (justify left))
-    )
-    (property "Value" "1.15M" (at 156.21 107.95 0)
-      (effects (font (size 1.27 1.27)) (justify left))
-    )
-    (property "Footprint" "Resistor_SMD:R_0603_1608Metric" (at 151.892 106.68 90)
-      (effects (font (size 1.27 1.27)) hide)
-    )
-    (property "Datasheet" "~" (at 153.67 106.68 0)
+  (symbol (lib_id "Device:R") (at 153.67 113.03 180) (unit 1)
+    (in_bom yes) (on_board yes) (dnp no) (fields_autoplaced)
+    (property "Reference" "R2" (at 156.21 111.76 0)
+      (effects (font (size 1.27 1.27)) (justify right))
+    )
+    (property "Value" "∞" (at 156.21 114.3 0)
+      (effects (font (size 1.27 1.27)) (justify right))
+    )
+    (property "Footprint" "Resistor_SMD:R_0603_1608Metric" (at 155.448 113.03 90)
+      (effects (font (size 1.27 1.27)) hide)
+    )
+    (property "Datasheet" "~" (at 153.67 113.03 0)
       (effects (font (size 1.27 1.27)) hide)
     )
@@
         )
       )
-      (project "DingLAB_miniPC_Power"
+      (project "DingLAB_miniPC_Power_Vertical"
         (path "/b2cfdd7f-acce-42ad-aab6-fa699ca2dca8"
           (reference "R2") (unit 1)
@@
       (effects (font (size 1.27 1.27)) (justify left))
     )
-    (property "Value" "MountingHole" (at 129.54 137.16 0)
+    (property "Value" "SMTSO3060CTJ" (at 129.54 137.16 0)
       (effects (font (size 1.27 1.27)) (justify left))
     )
@@
       (effects (font (size 1.27 1.27)) hide)
     )
-    (property "Datasheet" "~" (at 127 135.89 0)
-      (effects (font (size 1.27 1.27)) hide)
-    )
-    (instances
-      (project "DingLAB_miniPC_Power"
+    (property "Datasheet" "" (at 127 135.89 0)
+      (effects (font (size 1.27 1.27)) hide)
+    )
+    (property "lcsc" "C2915637" (at 127 135.89 0)
+      (effects (font (size 1.27 1.27)) hide)
+    )
+    (instances
+      (project "DingLAB_miniPC_Power_Vertical"
         (path "/b2cfdd7f-acce-42ad-aab6-fa699ca2dca8"
           (reference "H1") (unit 1)
@@
       (effects (font (size 1.27 1.27)))
     )
-    (property "Value" "KJB48xxSBO-10A" (at 121.92 99.06 0)
+    (property "Value" "KJB4815SBO-10A" (at 121.92 99.06 0)
       (effects (font (size 1.27 1.27)))
     )
@@
     (pin "7")
     (instances
-      (project "DingLAB_miniPC_Power"
+      (project "DingLAB_miniPC_Power_Vertical"
         (path "/b2cfdd7f-acce-42ad-aab6-fa699ca2dca8"
           (reference "U1") (unit 1)
@@
       (effects (font (size 1.27 1.27)) (justify left))
     )
-    (property "Value" "MountingHole" (at 129.54 142.24 0)
+    (property "Value" "SMTSO3060CTJ" (at 129.54 142.24 0)
       (effects (font (size 1.27 1.27)) (justify left))
     )
@@
       (effects (font (size 1.27 1.27)) hide)
     )
-    (instances
-      (project "DingLAB_miniPC_Power"
+    (property "lcsc" "C2915637" (at 127 140.97 0)
+      (effects (font (size 1.27 1.27)) hide)
+    )
+    (instances
+      (project "DingLAB_miniPC_Power_Vertical"
         (path "/b2cfdd7f-acce-42ad-aab6-fa699ca2dca8"
           (reference "H2") (unit 1)
@@
     )
   )
-  (symbol (lib_id "Device:R") (at 143.51 106.68 0) (unit 1)
-    (in_bom yes) (on_board yes) (dnp no) (fields_autoplaced)
-    (property "Reference" "R1" (at 146.05 105.41 0)
-      (effects (font (size 1.27 1.27)) (justify left))
-    )
-    (property "Value" "150k" (at 146.05 107.95 0)
-      (effects (font (size 1.27 1.27)) (justify left))
-    )
-    (property "Footprint" "Resistor_SMD:R_0603_1608Metric" (at 141.732 106.68 90)
-      (effects (font (size 1.27 1.27)) hide)
-    )
-    (property "Datasheet" "~" (at 143.51 106.68 0)
+  (symbol (lib_id "Device:R") (at 143.51 113.03 0) (unit 1)
+    (in_bom yes) (on_board yes) (dnp no) (fields_autoplaced)
+    (property "Reference" "R1" (at 146.05 111.76 0)
+      (effects (font (size 1.27 1.27)) (justify left))
+    )
+    (property "Value" "20k" (at 146.05 114.3 0)
+      (effects (font (size 1.27 1.27)) (justify left))
+    )
+    (property "Footprint" "Resistor_SMD:R_0603_1608Metric" (at 141.732 113.03 90)
+      (effects (font (size 1.27 1.27)) hide)
+    )
+    (property "Datasheet" "~" (at 143.51 113.03 0)
       (effects (font (size 1.27 1.27)) hide)
     )
@@
         )
       )
-      (project "DingLAB_miniPC_Power"
+      (project "DingLAB_miniPC_Power_Vertical"
         (path "/b2cfdd7f-acce-42ad-aab6-fa699ca2dca8"
           (reference "R1") (unit 1)
@@
         )
       )
-      (project "DingLAB_miniPC_Power"
+      (project "DingLAB_miniPC_Power_Vertical"
         (path "/b2cfdd7f-acce-42ad-aab6-fa699ca2dca8"
           (reference "J1") (unit 1)
@@
     (pin "1")
     (instances
-      (project "DingLAB_miniPC_Power"
+      (project "DingLAB_miniPC_Power_Vertical"
         (path "/b2cfdd7f-acce-42ad-aab6-fa699ca2dca8"
           (reference "#PWR01") (unit 1)
