File: DingLAB_miniPC_Power_Horizon_90.kicad_pcb (KiCad board)
At the start: 2 copper layers, 46.7 x 22.9 mm, 8 parts, among them J1 Conn_01x02_Pin, J2 Conn_01x02_Pin, U1 KJB48xxSBO-10A

Commit message: Update
Other:
- board text added: "MiniPC Power Horizen90 V1.0"
Changed lines of the file:
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@@
     (property "ki_keywords" "mounting hole")
     (attr smd)
-    (fp_text reference "H2" (at 0 -4.064 unlocked) (layer "F.SilkS")
+    (fp_text reference "H2" (at 0 -4.064 unlocked) (layer "F.SilkS") hide
         (effects (font (size 1 1) (thickness 0.1)))
     )
-    (fp_text value "MountingHole" (at 0 4.215 unlocked) (layer "F.Fab")
-        (effects (font (size 1 1) (thickness 0.15)))
-    )
-    (fp_text user "SMTSO3060CTJ" (at 0 5.715 unlocked) (layer "F.Fab")
+    (fp_text value "MountingHole" (at 0 4.215 unlocked) (layer "F.Fab") hide
         (effects (font (size 1 1) (thickness 0.15)))
     )
@@
     )
     (fp_text user "Ctrl" (at -11.90973 1.09699 unlocked) (layer "F.SilkS")
-        (effects (font (size 1.5 1.5) (thickness 0.3048)) (justify left bottom))
-    )
-    (fp_text user "KJB48_SBO-10A" (at -8.636 4.699 unlocked) (layer "F.SilkS")
         (effects (font (size 1.5 1.5) (thickness 0.3048)) (justify left bottom))
     )
@@
     (property "ki_keywords" "mounting hole")
     (attr smd)
-    (fp_text reference "H3" (at 0 -4.064 unlocked) (layer "F.SilkS")
+    (fp_text reference "H3" (at 0 -4.064 unlocked) (layer "F.SilkS") hide
         (effects (font (size 1 1) (thickness 0.1)))
     )
-    (fp_text value "MountingHole" (at 0 4.215 unlocked) (layer "F.Fab")
-        (effects (font (size 1 1) (thickness 0.15)))
-    )
-    (fp_text user "SMTSO3060CTJ" (at 0 5.715 unlocked) (layer "F.Fab")
+    (fp_text value "MountingHole" (at 0 4.215 unlocked) (layer "F.Fab") hide
         (effects (font (size 1 1) (thickness 0.15)))
     )
@@
     (property "ki_keywords" "connector")
     (attr through_hole)
-    (fp_text reference "J1" (at 2.5 -4 90) (layer "F.SilkS")
-        (effects (font (size 1 1) (thickness 0.15)))
-    )
-    (fp_text value "Conn_01x02_Pin" (at 2.5 4 90) (layer "F.Fab")
-        (effects (font (size 1 1) (thickness 0.15)))
-    )
-    (fp_text user "+" (at 9 0 90) (layer "F.SilkS")
-        (effects (font (size 1.5 1.5) (thickness 0.15)))
+    (fp_text reference "J1" (at 2.5 -4 90) (layer "F.SilkS") hide
+        (effects (font (size 1 1) (thickness 0.15)))
+    )
+    (fp_text value "Conn_01x02_Pin" (at 2.5 4 90) (layer "F.Fab") hide
+        (effects (font (size 1 1) (thickness 0.15)))
     )
     (fp_text user "-" (at -4 0 90) (layer "F.SilkS")
@@
     (property "ki_keywords" "connector")
     (attr through_hole)
-    (fp_text reference "J2" (at 2.5 -4 90) (layer "F.SilkS")
+    (fp_text reference "J2" (at 2.5 -4 90) (layer "F.SilkS") hide
         (effects (font (size 1 1) (thickness 0.15)))
     )
@@
     )
     (fp_text user "-" (at -4 0 90) (layer "F.SilkS")
-        (effects (font (size 1.5 1.5) (thickness 0.15)))
-    )
-    (fp_text user "+" (at 9 0 90) (layer "F.SilkS")
         (effects (font (size 1.5 1.5) (thickness 0.15)))
     )
@@
   (gr_rect (start 93.15 100) (end 139.85 122.86)
     (stroke (width 0.1) (type default)) (fill none) (layer "Edge.Cuts"))
+  (gr_text "MiniPC Power Horizen90 V1.0" (at 100.85 116.2) (layer "F.SilkS")
+    (effects (font (size 1 1) (thickness 0.15)) (justify left bottom))
+  )
   (segment (start 130.48 111.43) (end 129.09 111.43) (width 0.25) (layer "F.Cu") (net 5))
   (segment (start 127.77 112.75) (end 127.77 114.27) (width 0.25) (layer "F.Cu") (net 5))
